File: Library.kicad_blocks/nrf54l15-dk.kicad_block/nrf54l15-dk.kicad_sch (KiCad schematic)
At the start: 13 parts, among them J1 Conn_02x10_Odd_Even, J2 Conn_02x10_Odd_Even, J3 Conn_02x10_Odd_Even, J4 Conn_02x02_Odd_Even, J5 Conn_02x02_Odd_Even, J6 Conn_02x02_Odd_Even

Commit message: starting point of design block
Parts:
- renumbered H7 to H1, H8 to H2, H9 to H3, H10 to H4, H11 to H5, H12 to H6, J4 to J1, J5 to J2, J6 to J3, J1 to J4, J2 to J5, J3 to J6
