File: semtech_dev_board/54l15.kicad_sch (KiCad schematic)
At the start: 13 parts, among them J1 Conn_02x02_Odd_Even, J2 Conn_02x02_Odd_Even, J3 Conn_02x02_Odd_Even, J4 Conn_02x10_Odd_Even, J5 Conn_02x10_Odd_Even, J6 Conn_02x10_Odd_Even

Commit message: [fab] complete the design of semtech dev board
Connections:
- net +5V: now also J1.3 (Pin_3), J2.3 (Pin_3), J3.3 (Pin_3); no longer J1.1 (GND), J2.1 (Pin_1), J3.1 (Pin_1)
- net GND: now also J1.1 (GND), J2.1 (Pin_1), J3.1 (Pin_1); no longer J1.4 (Pin_4), J2.4 (Pin_4), J3.4 (Pin_4)
- net P2.00 renamed P2.00/QSPI_DIO3
- net P2.01 renamed P2.01/QSPI_CLK
- net P2.02 renamed P2.02/QSPI_DIO0
- net P2.03 renamed P2.03/QSPI_DIO2
- net P2.04 renamed P2.04/QSPI_DIO1
- net P2.05 renamed P2.05/QSPI_CS
Other:
- moved on the sheet: H1, H2, H3, H4, H5, H6, J2, J3, J5, J6, U1
